File: Hardware/MAX30105_Breakout.brd (EAGLE design)
At the start: 38.1 x 25.4 mm, 58 parts, among them J1 GATORGATOR_MINI, J2 GATORGATOR_MINI, J3 GATORGATOR_MINI, J4 GATORGATOR_MINI, J5 GATORGATOR_MINI, J6 GATORGATOR_MINI, J7 GATORGATOR_MINI, J8 GATORGATOR_MINI, Q1 200mA/50V, Q2 200mA/50V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

Commit message: forgot to save changes from review/checklist
Parts:
- added U$18: (no value), SparkFun-Aesthetics:ORDERING_INSTRUCTIONS
- LOGO1: value (none) -> SFE_LOGO_NAME_FLAME.1_INCH
- Q1, Q2: value 200mA/50V -> 220mA/50V/3.5Ω; device SparkFun-DiscreteSemi:SOT23-3@1 -> SparkFun-DiscreteSemi:SOT23-3
- STANDOFF2, STANDOFF3: value STAND-OFF -> STAND-OFFTIGHT; device SparkFun-Electromechanical:STAND-OFF -> SparkFun-Hardware:STAND-OFF-TIGHT
- U1: device SparkFun-PowerIC:SC70 -> SparkFun-IC-Power:SC70
- moved D1 2.54 mm to (29.2, 2.54)
- moved D2 1.27 mm to (19.1, 2.54)
- renumbered U$19 to LOGO1
Routing:
- net SCL: track 31.0 -> 33.5 mm
- net SDA: track 29.4 -> 30.5 mm
Other:
- board text added: "Black Gloss Soldermask"
- board text added: "v01"
- board text removed: "v10"
Changed lines of the file:
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@@
 <wire x1="38.1" y1="25.4" x2="38.1" y2="0" width="0.2032" layer="20"/>
 <wire x1="0" y1="0" x2="0" y2="25.4" width="0.2032" layer="20"/>
-<text x="20.701" y="0.635" size="1.27" layer="16" font="vector" ratio="20" rot="MR0">v10</text>
+<text x="20.701" y="0.635" size="1.27" layer="16" font="vector" ratio="20" rot="MR0">v01</text>
 <text x="27.94" y="-16.51" size="1.778" layer="51" font="vector" ratio="10">A. England</text>
 <text x="1.27" y="-3.81" size="1.778" layer="47" font="vector" ratio="15">All Dimensions in Inches</text>
 <dimension x1="38.1" y1="25.4" x2="0" y2="25.4" x3="19.05" y3="30.48" textsize="1.778" layer="47" unit="inch"/>
 <dimension x1="0" y1="25.4" x2="0" y2="0" x3="-5.08" y3="12.7" textsize="1.778" layer="47" unit="inch"/>
-<dimension x1="2.54" y1="22.86" x2="2.54" y2="2.54" x3="-1.27" y3="12.7" textsize="1.778" layer="47" unit="inch"/>
-<dimension x1="2.54" y1="22.86" x2="35.56" y2="22.86" x3="19.05" y3="26.67" textsize="1.778" layer="47" unit="inch"/>
+<text x="-7.62" y="-31.75" size="1.778" layer="51" font="vector" ratio="10">Black Gloss Soldermask</text>
 </plain>
 <attributes>
@@
 </autorouter>
 <elements>
-<element name="STANDOFF3" library="SparkFun-Electromechanical" package="STAND-OFF" value="STAND-OFF" x="2.54" y="12.7" smashed="yes"/>
-<element name="STANDOFF2" library="SparkFun-Electromechanical" package="STAND-OFF" value="STAND-OFF" x="35.56" y="12.7" smashed="yes"/>
+<element name="STANDOFF3" library="SparkFun-Hardware" package="STAND-OFF-TIGHT" value="STAND-OFFTIGHT" x="2.54" y="12.7" smashed="yes"/>
+<element name="STANDOFF2" library="SparkFun-Hardware" package="STAND-OFF-TIGHT" value="STAND-OFFTIGHT" x="35.56" y="12.7" smashed="yes"/>
 <element name="FID1" library="SparkFun-Aesthetics" package="FIDUCIAL-MICRO" value="FIDUCIALUFIDUCIAL" x="37.465" y="19.05" smashed="yes"/>
 <element name="FID2" library="SparkFun-Aesthetics" package="FIDUCIAL-MICRO" value="FIDUCIALUFIDUCIAL" x="0.635" y="6.35" smashed="yes" rot="MR0"/>
@@
 <attribute name="VALUE" x="22.987" y="14.605" size="0.6096" layer="27" font="vector" ratio="20" rot="R90" align="top-center"/>
 </element>
-<element name="Q1" library="SparkFun-DiscreteSemi" package="SOT23-3@1" value="200mA/50V" x="24.765" y="14.605" smashed="yes" rot="R270">
+<element name="Q1" library="SparkFun-DiscreteSemi" package="SOT23-3" value="220mA/50V/3.5Ω" x="24.765" y="14.605" smashed="yes" rot="R270">
 <attribute name="NAME" x="26.543" y="15.4305" size="0.4064" layer="25" rot="R270"/>
 <attribute name="PROD_ID" value="TRANS-00830" x="24.765" y="14.605" size="1.778" layer="27" font="vector" ratio="15" rot="R270" display="off"/>
-<attribute name="VALUE" x="24.5745" y="15.621" size="0.4064" layer="27" rot="R270"/>
-</element>
-<element name="Q2" library="SparkFun-DiscreteSemi" package="SOT23-3@1" value="200mA/50V" x="24.765" y="10.795" smashed="yes" rot="R270">
+<attribute name="VALUE" value="220mA/50V/3.5Ω" x="24.5745" y="15.621" size="0.4064" layer="27" rot="R270"/>
+</element>
+<element name="Q2" library="SparkFun-DiscreteSemi" package="SOT23-3" value="220mA/50V/3.5Ω" x="24.765" y="10.795" smashed="yes" rot="R270">
 <attribute name="NAME" x="26.543" y="11.6205" size="0.4064" layer="25" rot="R270"/>
 <attribute name="PROD_ID" value="TRANS-00830" x="24.765" y="10.795" size="1.778" layer="27" font="vector" ratio="15" rot="R270" display="off"/>
-<attribute name="VALUE" x="24.5745" y="11.811" size="0.4064" layer="27" rot="R270"/>
+<attribute name="VALUE" value="220mA/50V/3.5Ω" x="24.5745" y="11.811" size="0.4064" layer="27" rot="R270"/>
 </element>
 <element name="U2" library="SparkFun-Sensors" package="OLGA-14" value="30102" x="19.05" y="12.7" smashed="yes" rot="R180">
@@
 <attribute name="VALUE" x="19.05" y="15.748" size="0.6096" layer="27" font="vector" ratio="20" rot="R180" align="top-center"/>
 </element>
-<element name="FRAME1" library="SparkFun-Aesthetics" package="CREATIVE_COMMONS" value="FRAME-LETTER" x="-2.54" y="-16.51" smashed="yes"/>
+<element name="FRAME1" library="SparkFun-Aesthetics" package="CREATIVE_COMMONS" value="FRAME-LETTER" x="-2.54" y="-16.51" smashed="yes">
+<attribute name="DESIGNER" value="" x="-2.54" y="-16.51" size="1.778" layer="27" display="off"/>
+<attribute name="REV" value="" x="-2.54" y="-16.51" size="1.778" layer="27" display="off"/>
+</element>
 <element name="C1" library="SparkFun-Capacitors" package="0603" value="0.1uF" x="10.795" y="15.24" smashed="yes">
 <attribute name="NAME" x="9.906" y="16.002" size="0.4064" layer="25" font="vector"/>
@@
 <attribute name="VALUE" x="11.811" y="11.303" size="0.4064" layer="27" font="vector" rot="R180"/>
 </element>
-<element name="U1" library="SparkFun-PowerIC" package="SC70" value="1.8V/100mA" x="10.795" y="12.7" smashed="yes" rot="R180">
+<element name="U1" library="SparkFun-IC-Power" package="SC70" value="1.8V/100mA" x="10.795" y="12.7" smashed="yes" rot="R180">
 <attribute name="NAME" x="11.684" y="11.176" size="0.4064" layer="25" rot="R180"/>
 <attribute name="PROD_ID" value="VREG-08428" x="10.795" y="12.7" size="1.778" layer="27" font="vector" ratio="15" rot="R180" display="off"/>
@@
 <element name="U$15" library="buzzard_labels (2)" package="SDA2" value="" x="26.543" y="8.001" smashed="yes" rot="MR0"/>
 <element name="U$16" library="buzzard_labels (2)" package="SCL1" value="" x="36.576" y="8.001" smashed="yes" rot="MR0"/>
-<element name="D1" library="SparkFun-DiscreteSemi" package="SOD-323" value="3.6V" x="29.21" y="5.08" smashed="yes" rot="R270">
-<attribute name="NAME" x="29.972" y="5.08" size="0.6096" layer="25" font="vector" ratio="20" rot="R270" align="bottom-center"/>
-<attribute name="PROD_ID" value="DIO-08199" x="29.21" y="5.08" size="1.778" layer="27" rot="R270" display="off"/>
-<attribute name="VALUE" x="28.448" y="5.08" size="0.6096" layer="27" font="vector" ratio="20" rot="R270" align="top-center"/>
-</element>
-<element name="D2" library="SparkFun-DiscreteSemi" package="SOD-323" value="3.6V" x="19.05" y="3.81" smashed="yes" rot="R270">
-<attribute name="NAME" x="19.812" y="3.81" size="0.6096" layer="25" font="vector" ratio="20" rot="R270" align="bottom-center"/>
-<attribute name="PROD_ID" value="DIO-08199" x="19.05" y="3.81" size="1.778" layer="27" rot="R270" display="off"/>
-<attribute name="VALUE" x="18.288" y="3.81" size="0.6096" layer="27" font="vector" ratio="20" rot="R270" align="top-center"/>
+<element name="D1" library="SparkFun-DiscreteSemi" package="SOD-323" value="3.6V" x="29.21" y="2.54" smashed="yes" rot="R270">
+<attribute name="NAME" x="29.972" y="2.54" size="0.6096" layer="25" font="vector" ratio="20" rot="R270" align="bottom-center"/>
+<attribute name="PROD_ID" value="DIO-08199" x="29.21" y="2.54" size="1.778" layer="27" rot="R270" display="off"/>
+<attribute name="VALUE" x="28.448" y="2.54" size="0.6096" layer="27" font="vector" ratio="20" rot="R270" align="top-center"/>
+</element>
+<element name="D2" library="SparkFun-DiscreteSemi" package="SOD-323" value="3.6V" x="19.05" y="2.54" smashed="yes" rot="R270">
+<attribute name="NAME" x="19.812" y="2.54" size="0.6096" layer="25" font="vector" ratio="20" rot="R270" align="bottom-center"/>
+<attribute name="PROD_ID" value="DIO-08199" x="19.05" y="2.54" size="1.778" layer="27" rot="R270" display="off"/>
+<attribute name="VALUE" x="18.288" y="2.54" size="0.6096" layer="27" font="vector" ratio="20" rot="R270" align="top-center"/>
 </element>
 <element name="D3" library="SparkFun-DiscreteSemi" package="SOD-323" value="3.6V" x="10.287" y="7.366" smashed="yes" rot="R270">
@@
 </element>
 <element name="U$17" library="SparkFun-Aesthetics" package="SFE_LOGO_FLAME_.2" value="" x="31.242" y="12.573"/>
-<element name="U$19" library="SparkFun-Aesthetics" package="SFE_LOGO_NAME_FLAME_.1" value="" x="19.05" y="15.24" rot="MR0"/>
 <element name="U$20" library="buzzard_labels (4)" package="GATOR#PARTICLE2" value="" x="24.765" y="12.827" rot="MR0"/>
 <element name="U$21" library="GatorBit_Final_for_Silk#01#png (3)" package="GATORBIT_FINAL_FOR_SILK#01#PNG" value="" x="18.923" y="10.16" rot="MR0"/>
@@
 </element>
 <element name="U$22" library="buzzard_labels (5)" package="PWR0" value="" x="21.59" y="17.399" rot="R180"/>
+<element name="LOGO1" library="SparkFun-Aesthetics" package="SFE_LOGO_NAME_FLAME_.1" value="SFE_LOGO_NAME_FLAME.1_INCH" x="19.05" y="15.24" rot="MR0"/>
+<element name="U$18" library="SparkFun-Aesthetics" package="ORDERING_INSTRUCTIONS" value="" x="-8.89" y="-20.32"/>
 </elements>
 <signals>
@@
 <contactref element="J3" pad="P$2"/>
 <contactref element="J7" pad="P$2"/>
-<wire x1="25.865" y1="14.605" x2="26.035" y2="14.605" width="0.2032" layer="1"/>
 <wire x1="25.865" y1="14.605" x2="25.865" y2="12.149" width="0.2032" layer="1"/>
 <wire x1="25.865" y1="14.605" x2="25.865" y2="15.494" width="0.2032" layer="1"/>
@@
 <wire x1="24.765" y1="11.049" x2="24.765" y2="8.255" width="0.2032" layer="1"/>
 <contactref element="D2" pad="C"/>
-<wire x1="19.05" y1="4.96" x2="19.05" y2="6.985" width="0.2032" layer="1"/>
+<wire x1="19.05" y1="3.69" x2="19.05" y2="6.985" width="0.2032" layer="1"/>
 <wire x1="19.05" y1="6.985" x2="19.685" y2="7.62" width="0.2032" layer="1"/>
 <wire x1="19.685" y1="7.62" x2="24.13" y2="7.62" width="0.2032" layer="1"/>
@@
 <wire x1="30.265" y1="9.945" x2="31.75" y2="11.43" width="0.2032" layer="1"/>
 <contactref element="D1" pad="C"/>
-<wire x1="29.21" y1="6.23" x2="29.21" y2="9.945" width="0.2032" layer="1"/>
+<wire x1="29.21" y1="3.69" x2="29.21" y2="9.945" width="0.2032" layer="1"/>
 </signal>
 <signal name="N$30">
@@
 <wire x1="22.225" y1="13.755" x2="23.665" y2="13.755" width="0.2032" layer="1"/>
 <wire x1="23.665" y1="13.755" x2="23.765" y2="13.655" width="0.2032" layer="1"/>
-<wire x1="20.25" y1="11.9" x2="20.32" y2="11.9" width="0.2032" layer="1"/>
 <wire x1="21.59" y1="12.7" x2="21.971" y2="12.7" width="0.2032" layer="1"/>
 <wire x1="21.971" y1="12.7" x2="22.225" y2="12.954" width="0.2032" layer="1"/>
