File: Hardware/GatorParticle.sch (EAGLE design)
At the start: 38 parts, among them J1 GATORGATOR_MINI, J2 GATORGATOR_MINI, J3 GATORGATOR_MINI, J4 GATORGATOR_MINI, J5 GATORGATOR_MINI, J6 GATORGATOR_MINI, J7 GATORGATOR_MINI, J8 GATORGATOR_MINI, Q1 220mA/50V/3.5Ω, Q2 220mA/50V/3.5Ω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

Commit message: engineer run of checklist
Other:
- note added: "7-Bit Unshifted I2C Address: 0x57"
- note added: "Connections"
- note added: "Input Voltage: 3.3-7V"
- note added: "Logic Level Conversion"
- note added: "MAX30102 Particle Sensor"
- note added: "v10"
- note removed: "7-Bit I2C: 0x57"
- note removed: "Interface and Logic Conversion"
- note removed: "Sensor"
- note removed: "VIN: 3-7V"
- note removed: "v01"
- moved on the sheet: D1, D2, D3, D4, J1, J2, J3, J4, J5, J6, J7, J8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
