File: Hardware/GatorParticle.brd (EAGLE design)
At the start: 38.1 x 25.4 mm, 59 parts, among them J1 GATORGATOR_MINI, J2 GATORGATOR_MINI, J3 GATORGATOR_MINI, J4 GATORGATOR_MINI, J5 GATORGATOR_MINI, J6 GATORGATOR_MINI, J7 GATORGATOR_MINI, J8 GATORGATOR_MINI, Q1 220mA/50V/3.5Ω, Q2 220mA/50V/3.5Ω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

Commit message: Post checklist changes
Parts:
- moved LOGO2 1.27 mm to (19.1, 3.17)
Changed lines of the file:
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@@
 <attribute name="VALUE" x="14.478" y="11.684" size="0.4064" layer="27" font="vector" rot="R90"/>
 </element>
-<element name="LOGO2" library="SparkFun-Aesthetics" package="OSHW-LOGO-S" value="OSHW-LOGOS" x="19.05" y="1.905" smashed="yes" rot="MR0"/>
+<element name="LOGO2" library="SparkFun-Aesthetics" package="OSHW-LOGO-S" value="OSHW-LOGOS" x="19.05" y="3.175" smashed="yes" rot="MR0"/>
 <element name="R8" library="SparkFun-Resistors" package="0603" value="2.2k" x="22.225" y="10.795" smashed="yes" rot="R90">
 <attribute name="NAME" x="21.463" y="10.795" size="0.6096" layer="25" font="vector" ratio="20" rot="R90" align="bottom-center"/>

Commit message: engineer run of checklist
Parts:
- removed U$20: (no value), buzzard_labels (4):GATOR#PARTICLE2
- added U$19: (no value), buzzard_labels (13):PWR0
- U$22: device buzzard_labels (5):PWR0 -> buzzard_labels (14):GATOR#PARTICLE0
- moved U$22 8.43 mm to (28.8, 13.1), flipped to the bottom, turned to 0 degrees
- moved TP1 0.63 mm to (14.0, 10.2)
- moved D4 0.63 mm to (19.1, 19.1)
- moved U$17 0.36 mm to (31.0, 12.8), turned to 180 degrees
- moved U$16 0.13 mm to (36.4, 8.00)
- moved U$7 0.13 mm to (21.8, 17.4)
- moved U$8 0.13 mm to (32.1, 17.4)
- moved U$5 0.13 mm to (1.40, 17.5)
- moved U$9 0.13 mm to (6.22, 17.5)
- moved U$10 0.13 mm to (16.3, 17.4)
- moved U$14 0.13 mm to (16.3, 8.00)
- moved U$15 0.13 mm to (26.4, 8.00)
Routing:
- net N$3: track 2.69 -> 3.32 mm
- net 3.3V: track 55.4 -> 54.7 mm
Other:
- board text added: "v10"
- board text removed: "v01"

Commit message: qc double check changes
Routing:
- net GND: vias 6 -> 8
Changed lines of the file:
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@@
 <wire x1="20.25" y1="12.7" x2="20.701" y2="12.7" width="0.2032" layer="1"/>
 <wire x1="20.701" y1="12.7" x2="21.336" y2="13.335" width="0.2032" layer="1"/>
-<via x="19.05" y="12.192" extent="1-16" drill="0.381"/>
+<via x="19.05" y="11.049" extent="1-16" drill="0.381"/>
 <via x="8.509" y="10.541" extent="1-16" drill="0.381"/>
-<via x="19.05" y="14.732" extent="1-16" drill="0.381"/>
+<via x="19.05" y="14.478" extent="1-16" drill="0.381"/>
 <contactref element="D1" pad="A"/>
 <contactref element="D2" pad="A"/>
@@
 <contactref element="R3" pad="1"/>
 <contactref element="R4" pad="1"/>
+<via x="12.827" y="9.525" extent="1-16" drill="0.381"/>
+<via x="8.255" y="15.748" extent="1-16" drill="0.381"/>
 </signal>
 <signal name="SDA">
@@
 <wire x1="25.908" y1="13.462" x2="19.05" y2="13.462" width="0.2032" layer="16"/>
 <via x="19.05" y="13.462" extent="1-16" drill="0.381"/>
-<wire x1="19.05" y1="13.462" x2="19.012" y2="13.5" width="0.2032" layer="1"/>
-<wire x1="19.012" y1="13.5" x2="17.85" y2="13.5" width="0.2032" layer="1"/>
+<wire x1="18.923" y1="13.462" x2="18.885" y2="13.5" width="0.2032" layer="1"/>
+<wire x1="18.885" y1="13.5" x2="17.85" y2="13.5" width="0.2032" layer="1"/>
 <wire x1="9.945" y1="15.24" x2="9.945" y2="14.439" width="0.2032" layer="1"/>
 <contactref element="R1" pad="2"/>
@@
 <contactref element="R5" pad="2"/>
 <wire x1="15.24" y1="12.715" x2="15.24" y2="13.55" width="0.2032" layer="1"/>
+<wire x1="19.05" y1="13.462" x2="18.923" y2="13.462" width="0.2032" layer="1"/>
 </signal>
 <signal name="1.8V">
@@
 <wire x1="24.445" y1="11.745" x2="23.765" y2="11.745" width="0.2032" layer="1"/>
 <wire x1="24.765" y1="12.065" x2="24.445" y2="11.745" width="0.2032" layer="1"/>
-<wire x1="16.383" y1="11.811" x2="16.383" y2="14.4833" width="0.2032" layer="16"/>
-<wire x1="16.383" y1="14.4833" x2="16.000134375" y2="14.866165625" width="0.2032" layer="16"/>
-<via x="16.000134375" y="14.866165625" extent="1-16" drill="0.381"/>
-<wire x1="16.000134375" y1="14.866165625" x2="16.000134375" y2="16.000134375" width="0.2032" layer="1"/>
-<wire x1="16.000134375" y1="16.000134375" x2="16.51" y2="16.51" width="0.2032" layer="1"/>
+<wire x1="16.383" y1="11.811" x2="16.383" y2="14.7373" width="0.2032" layer="16"/>
+<wire x1="16.383" y1="14.7373" x2="15.873134375" y2="15.247165625" width="0.2032" layer="16"/>
+<via x="15.873134375" y="15.247165625" extent="1-16" drill="0.381"/>
+<wire x1="15.873134375" y1="15.247165625" x2="15.873134375" y2="15.873134375" width="0.2032" layer="1"/>
+<wire x1="15.873134375" y1="15.873134375" x2="16.51" y2="16.51" width="0.2032" layer="1"/>
 <wire x1="16.51" y1="16.51" x2="24.13" y2="16.51" width="0.2032" layer="1"/>
 <wire x1="24.13" y1="16.51" x2="24.765" y2="15.875" width="0.2032" layer="1"/>
